File: VGA.kicad_sch (KiCad schematic)
At the start: 2 parts

Commit message: だいたい完成
Parts:
- added C1: C, Capacitor_THT:CP_Radial_D5.0mm_P2.50mm, symbol Device:C_Polarized
- added C10, C11, C12, C13, C14, C15, C16, C2, C3, C4, C5, C6, C7, C8, C9: C, Capacitor_THT:C_Disc_D7.0mm_W2.5mm_P5.00mm, symbol Device:C
- added U14: 74HC02, Package_DIP:DIP-14_W7.62mm, symbol 74xx:74HC02
- U1, U2: renamed from U?; footprint (none) -> Package_DIP:DIP-14_W7.62mm
Connections:
- net GND: now also C1.2, C10.2, C11.2, C12.2, C13.2, C14.2, C15.2, C16.2, C2.2, C3.2, C4.2, C5.2, C6.2, C7.2, C8.2, C9.2, U14.7 (GND)
- net VCC: now also C1.1, C10.1, C11.1, C12.1, C13.1, C14.1, C15.1, C16.1, C2.1, C3.1, C4.1, C5.1, C6.1, C7.1, C8.1, C9.1, U14.14 (VCC)

Commit message: 信号生成部設計完了
Parts:
- added C1: C, Capacitor_THT:C_Disc_D7.0mm_W2.5mm_P5.00mm, symbol Device:C
- added H1, H2, H3, H4: MountingHole_Pad, MountingHole:MountingHole_3mm_Pad, symbol Mechanical:MountingHole_Pad
- renumbered C1 to C19, U14 to U3
Connections:
- net GND: now also C1.2, H1.1, H2.1, H3.1, H4.1
- net VCC: now also C1.1
Other:
- moved on the sheet: C19

Commit message: 完成版
Parts:
- added D1: LED, LED_THT:LED_D3.0mm, symbol Device:LED
- added R8: R, Resistor_SMD:R_0603_1608Metric_Pad0.98x0.95mm_HandSolder, symbol Device:R
Connections:
- net GND: now also R8.2
- net VCC: now also D1.2 (A)
- new net: D1.1 (K), R8.1
Changed lines of the file:
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@@
   (junction (at 180.34 111.76) (diameter 0) (color 0 0 0 0)
   )
+  (wire (pts (xy 227.33 50.8) (xy 233.68 50.8))
+    (stroke (width 0) (type default) (color 0 0 0 0))
+  )
   (wire (pts (xy 198.12 88.9) (xy 208.28 88.9))
     (stroke (width 0) (type default) (color 0 0 0 0))
@@
     (stroke (width 0) (type default) (color 0 0 0 0))
   )
+  (wire (pts (xy 233.68 49.53) (xy 233.68 50.8))
+    (stroke (width 0) (type default) (color 0 0 0 0))
+  )
   (wire (pts (xy 153.67 96.52) (xy 144.78 96.52))
     (stroke (width 0) (type default) (color 0 0 0 0))
@@
     (stroke (width 0) (type default) (color 0 0 0 0))
   )
+  (wire (pts (xy 212.09 59.69) (xy 212.09 58.42))
+    (stroke (width 0) (type default) (color 0 0 0 0))
+  )
   (wire (pts (xy 180.34 88.9) (xy 189.23 88.9))
     (stroke (width 0) (type default) (color 0 0 0 0))
@@
   )
   (wire (pts (xy 162.56 104.14) (xy 171.45 104.14))
+    (stroke (width 0) (type default) (color 0 0 0 0))
+  )
+  (wire (pts (xy 212.09 50.8) (xy 219.71 50.8))
     (stroke (width 0) (type default) (color 0 0 0 0))
   )
@@
     )
     (pin "1")
+  )
+  (symbol (lib_id "Device:LED") (at 223.52 50.8 0) (unit 1)
+    (in_bom yes) (on_board yes) (fields_autoplaced)
+    (property "Reference" "D1" (id 0) (at 221.9325 44.45 0))
+    (property "Value" "LED" (id 1) (at 221.9325 46.99 0))
+    (property "Footprint" "LED_THT:LED_D3.0mm" (id 2) (at 223.52 50.8 0)
+      (effects (font (size 1.27 1.27)) hide)
+    )
+    (property "Datasheet" "~" (id 3) (at 223.52 50.8 0)
+      (effects (font (size 1.27 1.27)) hide)
+    )
+    (pin "1")
+    (pin "2")
   )
   (symbol (lib_id "Device:C") (at 144.78 107.95 0) (unit 1)
@@
     (pin "1")
   )
+  (symbol (lib_id "Device:R") (at 212.09 54.61 0) (unit 1)
+    (in_bom yes) (on_board yes) (fields_autoplaced)
+    (property "Reference" "R8" (id 0) (at 214.63 53.3399 0)
+      (effects (font (size 1.27 1.27)) (justify left))
+    )
+    (property "Value" "R" (id 1) (at 214.63 55.8799 0)
+      (effects (font (size 1.27 1.27)) (justify left))
+    )
+    (property "Footprint" "Resistor_SMD:R_0603_1608Metric_Pad0.98x0.95mm_HandSolder" (id 2) (at 210.312 54.61 90)
+      (effects (font (size 1.27 1.27)) hide)
+    )
+    (property "Datasheet" "~" (id 3) (at 212.09 54.61 0)
+      (effects (font (size 1.27 1.27)) hide)
+    )
+    (pin "1")
+    (pin "2")
+  )
   (symbol (lib_id "power:VCC") (at 208.28 86.36 0) (unit 1)
     (in_bom yes) (on_board yes)
@@
     )
     (property "Datasheet" "" (id 3) (at 140.97 33.02 0)
+      (effects (font (size 1.27 1.27)) hide)
+    )
+    (pin "1")
+  )
+  (symbol (lib_id "power:GND") (at 212.09 59.69 0) (unit 1)
+    (in_bom yes) (on_board yes)
+    (property "Reference" "#PWR068" (id 0) (at 212.09 66.04 0)
+      (effects (font (size 1.27 1.27)) hide)
+    )
+    (property "Value" "GND" (id 1) (at 208.28 59.69 0))
+    (property "Footprint" "" (id 2) (at 212.09 59.69 0)
+      (effects (font (size 1.27 1.27)) hide)
+    )
+    (property "Datasheet" "" (id 3) (at 212.09 59.69 0)
       (effects (font (size 1.27 1.27)) hide)
     )
@@
     (pin "1")
   )
+  (symbol (lib_id "power:VCC") (at 233.68 49.53 0) (unit 1)
+    (in_bom yes) (on_board yes)
+    (property "Reference" "#PWR067" (id 0) (at 233.68 53.34 0)
+      (effects (font (size 1.27 1.27)) hide)
+    )
+    (property "Value" "VCC" (id 1) (at 229.87 48.26 0))
+    (property "Footprint" "" (id 2) (at 233.68 49.53 0)
+      (effects (font (size 1.27 1.27)) hide)
+    )
+    (property "Datasheet" "" (id 3) (at 233.68 49.53 0)
+      (effects (font (size 1.27 1.27)) hide)
+    )
+    (pin "1")
+  )
   (symbol (lib_id "Device:C") (at 171.45 107.95 0) (unit 1)
     (in_bom yes) (on_board yes) (fields_autoplaced)
@@
       (reference "#PWR052") (unit 1) (value "VCC") (footprint "")
     )
-    (path "/6bda3ce2-36c6-4424-8c17-cd51083511b5/e23a20f5-6b7a-4e93-b1fa-2026bad23a8d"
-      (reference "#PWR053") (unit 1) (value "VCC") (footprint "")
-    )
     (path "/6bda3ce2-36c6-4424-8c17-cd51083511b5/b9400199-61a6-4dde-9fa0-f71cfad6bd53"
       (reference "#PWR054") (unit 1) (value "GND") (footprint "")
@@
       (reference "#PWR063") (unit 1) (value "GND") (footprint "")
     )
+    (path "/3206bd33-f28a-4398-afb1-82a1c4945b28/6e82e81e-c3c8-40d6-b63a-cfc8f0c78dbf"
+      (reference "#PWR064") (unit 1) (value "VCC") (footprint "")
+    )
+    (path "/3206bd33-f28a-4398-afb1-82a1c4945b28/e25ec5c4-f871-449a-8f19-1de46c0dce9a"
+      (reference "#PWR065") (unit 1) (value "GND") (footprint "")
+    )
+    (path "/3206bd33-f28a-4398-afb1-82a1c4945b28/7bdf5066-efc0-43b9-b258-be3fc0d74b08"
+      (reference "#PWR066") (unit 1) (value "VCC") (footprint "")
+    )
+    (path "/9f9a205c-0db7-4883-ad26-b1b3e8f7c950"
+      (reference "#PWR067") (unit 1) (value "VCC") (footprint "")
+    )
+    (path "/51f6670e-d6b1-490e-ac8b-316d8ef582b1"
+      (reference "#PWR068") (unit 1) (value "GND") (footprint "")
+    )
+    (path "/6bda3ce2-36c6-4424-8c17-cd51083511b5/d7550967-22d2-494b-ae5e-7c5cc26134bb"
+      (reference "#PWR069") (unit 1) (value "VCC") (footprint "")
+    )
+    (path "/6bda3ce2-36c6-4424-8c17-cd51083511b5/716a9a6e-0c9e-4760-ba95-2e2c0b2bc1bd"
+      (reference "#PWR070") (unit 1) (value "VCC") (footprint "")
+    )
     (path "/ee2e6994-68b1-458f-87ee-c3306ff72b68"
       (reference "C1") (unit 1) (value "C") (footprint "Capacitor_THT:C_Disc_D7.0mm_W2.5mm_P5.00mm")
@@
       (reference "C19") (unit 1) (value "C") (footprint "Capacitor_THT:CP_Radial_D5.0mm_P2.50mm")
     )
+    (path "/09ae951c-4b14-42e4-9f4a-b7b1369a7424"
+      (reference "D1") (unit 1) (value "LED") (footprint "LED_THT:LED_D3.0mm")
+    )
+    (path "/6bda3ce2-36c6-4424-8c17-cd51083511b5/ebcf2c3f-c375-4dc6-a718-0bf1ce6bbaba"
+      (reference "D2") (unit 1) (value "LED") (footprint "LED_THT:LED_D3.0mm")
+    )
+    (path "/6bda3ce2-36c6-4424-8c17-cd51083511b5/c0a52e96-db7d-4a8a-8795-d8f25d9066d1"
+      (reference "D3") (unit 1) (value "LED") (footprint "LED_THT:LED_D3.0mm")
+    )
     (path "/91f13b4c-e5e9-4c74-be19-46e859b90c80"
       (reference "H1") (unit 1) (value "MountingHole_Pad") (footprint "MountingHole:MountingHole_3mm_Pad")
@@
     )
     (path "/3206bd33-f28a-4398-afb1-82a1c4945b28/17a6c8ee-1411-4597-88c8-5e9c3fdcff62"
-      (reference "JP1") (unit 1) (value "Jumper_3_Bridged12") (footprint "Jumper:SolderJumper-3_P1.3mm_Bridged12_Pad1.0x1.5mm")
+      (reference "JP1") (unit 1) (value "Jumper_3_Bridged12") (footprint "Jumper:SolderJumper-3_P1.3mm_Open_RoundedPad1.0x1.5mm")
     )
     (path "/3206bd33-f28a-4398-afb1-82a1c4945b28/10437ae3-55bf-41d0-9868-e6cd7d9bd112"
@@
       (reference "R7") (unit 1) (value "470") (footprint "Resistor_SMD:R_0603_1608Metric_Pad0.98x0.95mm_HandSolder")
     )
+    (path "/2c3e9aec-566a-4063-a731-6f3aa97d23c8"
+      (reference "R8") (unit 1) (value "R") (footprint "Resistor_SMD:R_0603_1608Metric_Pad0.98x0.95mm_HandSolder")
+    )
+    (path "/6bda3ce2-36c6-4424-8c17-cd51083511b5/2e42870b-65e0-4bcb-a5fb-950f1498bd83"
+      (reference "R9") (unit 1) (value "R") (footprint "Resistor_SMD:R_0603_1608Metric_Pad0.98x0.95mm_HandSolder")
+    )
+    (path "/6bda3ce2-36c6-4424-8c17-cd51083511b5/0287557c-0a13-42de-814d-eeeb8063791e"
+      (reference "R10") (unit 1) (value "R") (footprint "Resistor_SMD:R_0603_1608Metric_Pad0.98x0.95mm_HandSolder")
+    )
+    (path "/3206bd33-f28a-4398-afb1-82a1c4945b28/6521c893-b89a-4402-9a20-340b7c1794d6"
+      (reference "RN1") (unit 1) (value "R_Network04") (footprint "Resistor_THT:R_Array_SIP5")
+    )
     (path "/3206bd33-f28a-4398-afb1-82a1c4945b28/5a4eac72-4486-4334-8fb4-9898088393ab"
-      (reference "SW1") (unit 1) (value "SW_DIP_x03") (footprint "Button_Switch_THT:SW_DIP_SPSTx03_Slide_9.78x9.8mm_W7.62mm_P2.54mm")
+      (reference "SW1") (unit 1) (value "SW_DIP_x03") (footprint "Button_Switch_THT:SW_DIP_SPSTx03_Piano_10.8x9.18mm_W7.62mm_P2.54mm")
+    )
+    (path "/3206bd33-f28a-4398-afb1-82a1c4945b28/83a1fdd5-863f-4e82-9d5a-d74d63c2a36e"
+      (reference "SW2") (unit 1) (value "SW_DIP_x04") (footprint "Button_Switch_THT:SW_DIP_SPSTx04_Piano_10.8x11.72mm_W7.62mm_P2.54mm")
+    )
+    (path "/3206bd33-f28a-4398-afb1-82a1c4945b28/35df7212-8b11-4e4f-8855-ec1193da5ab3"
+      (reference "TP1") (unit 1) (value "TestPoint") (footprint "TestPoint:TestPoint_THTPad_D1.0mm_Drill0.5mm")
+    )
+    (path "/3206bd33-f28a-4398-afb1-82a1c4945b28/ce6094bd-a36c-416a-8b4c-19b11b0f7f96"
+      (reference "TP2") (unit 1) (value "TestPoint") (footprint "TestPoint:TestPoint_THTPad_D1.0mm_Drill0.5mm")
+    )
+    (path "/3206bd33-f28a-4398-afb1-82a1c4945b28/a7c8abd0-8da8-4e89-8a9c-cdaf9bf663aa"
+      (reference "TP3") (unit 1) (value "TestPoint") (footprint "TestPoint:TestPoint_THTPad_D1.0mm_Drill0.5mm")
     )
     (path "/3206bd33-f28a-4398-afb1-82a1c4945b28/4251262b-4b2b-41bc-a446-dec12741dcdb"
